File: PCB/Main/UGC_Main.kicad_sch (KiCad schematic)
At the start: 19 parts, among them J1 Rumble, J2 LT, J3 RT, J4 UJ31-CH-G1-SMT-TR, SW1 SW_Push, SW10 SW_Push, SW11 SW_Push, SW12 SW_Push, SW13 SW_Push, SW2 SW_Push, SW3 SW_Push, SW4 SW_Push, SW5 SW_Push, SW6 GL18_SW, SW7 SW_Push, SW8 SW_Push, SW9 TS09-63-25-R-260-SMT

Commit message: Update shell and PCB
Parts:
- added J10, J11, J12, J5, J6, J7, J8, J9: Conn_01x01_Pin, hhl:YZ72015053P-01, symbol Connector:Conn_01x01_Pin
- added U1: ESP32-PICO-MINI-02, hhl:MODULE_ESP32-PICO-MINI-02, symbol hhl:ESP32-PICO-MINI-02
Connections:
- new net: U1.1 (GND), U1.11 (GND), U1.14 (GND), U1.2 (GND), U1.36 (GND), U1.37 (GND), U1.38 (GND), U1.39 (GND), U1.40 (GND), U1.41 (GND), U1.42 (GND), U1.43 (GND), U1.44 (GND), U1.45 (GND), U1.46 (GND), U1.47 (GND), U1.48 (GND), U1.49 (GND), U1.50 (GND), U1.51 (GND), U1.52 (GND), U1.53 (GND), U1.54 (GND), U1.55 (GND), U1.56 (GND), U1.57 (GND), U1.58 (GND), U1.59 (GND), U1.60 (GND), U1.61 (GND)
- new net: U1.25 (NC), U1.32 (NC)
