File: PCB/Trigger/UGC_Trigger.kicad_pcb (KiCad board)
At the start: 2 copper layers, 9.2 x 18.5 mm, 3 parts, among them J1 Conn_01x01_Pin, J2 Conn_01x01_Pin, SW1 SW_Push

Commit message: Update shell and PCB
Parts:
- SW1: footprint hhl:progcc_bpad -> hhl:snes_pad
- moved SW1 0.24 mm to (278.9, 159.0)
Routing:
- net Net-(J2-Pin_1): track 19.4 -> 22.7 mm
- net Net-(J1-Pin_1): track 10.0 -> 12.7 mm
Other:
- board size 9.2 x 18.5 mm -> 9.3 x 19.1 mm
