File: PCB/Trigger/UGC_Trigger.kicad_sch (KiCad schematic)
At the start: 3 parts, among them J1 Conn_01x01_Pin, J2 Conn_01x01_Pin, SW1 SW_Push

Commit message: Update shell and PCB
Parts:
- SW1: footprint hhl:progcc_bpad -> hhl:snes_pad
Changed lines of the file:
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@@
       (effects (font (size 1.27 1.27)))
     )
-    (property "Footprint" "hhl:progcc_bpad" (at 223.52 149.86 0)
+    (property "Footprint" "hhl:snes_pad" (at 223.52 149.86 0)
       (effects (font (size 1.27 1.27)) hide)
     )
